Commit message: wip_with_gazebo

File: dts_stack/urdf/ackermannRobot/camera.xacro (robot description, xacro)
@@ -8,25 +8,26 @@
       <material name="silver"/>
     </visual>
-    <xacro:inertial_box mass="0.1" x="0.025" y="0.125" z="0.03">
+    <xacro:box_inertial_w_origin mass="0.1" length="0.025" breadth="0.125" height="0.03">
     <origin xyz="0 0 0" rpy="0 0 0"/>
-  </xacro:inertial_box>
+  </xacro:box_inertial_w_origin>
   </link>
   <joint name="camera_joint" type="fixed">
-    <parent link="base_link"/>
+    <parent link="chassis_link"/>
     <child link="camera_link"/>
-    <origin xyz="0.155 0 ${base_height/2 + 0.05}" rpy="0 0 0"/>
+    <origin xyz="0.155 0 ${chassis_height/2 + 0.015}" rpy="0 0 0"/>
   </joint>
-  <link name="camera_link_optical"></link>
+  <!-- <link name="camera_link_optical"></link>
   <joint name="camera_optical_joint" type="fixed">
     <parent link="camera_link"/>
     <child link="camera_link_optical"/>
     <origin xyz="0 0 0" rpy="${-pi/2} 0 ${-pi/2}"/>
-  </joint>
+  </joint> -->
   <gazebo reference="camera_link">
-    <material>Gazebo/Black</material>
+    <material>Gazebo/Silver</material>
     <sensor name="camera" type="camera">
       <pose> 0 0 0 0 0 0 </pose>
       <visualize>true</visualize>
       <update_rate>10</update_rate>
+      <topic>camera</topic>
       <camera>
         <horizontal_fov>1.089</horizontal_fov>

File: dts_stack/urdf/ackermannRobot/depth_camera.xacro (robot description, xacro)
@@ -1,42 +1,37 @@
 <?xml version="1.0"?>
 <robot xmlns:xacro="http://www.ros.org/wiki/xacro" >
-  <link name="camera_link">
+  <link name="depth_camera_link">
     <visual>
       <geometry>
-        <box size="0.01 0.03 0.03"/>
+        <box size="0.025 0.125 0.03"/>
       </geometry>
-      <material name="red"/>
+      <material name="silver"/>
     </visual>
-    <xacro:inertial_box mass="0.1" x="0.01" y="0.03" z="0.03">
+    <xacro:box_inertial_w_origin mass="0.1" length="0.025" breadth="0.125" height="0.03">
     <origin xyz="0 0 0" rpy="0 0 0"/>
-  </xacro:inertial_box>
+  </xacro:box_inertial_w_origin>
   </link>
-  <joint name="camera_joint" type="fixed">
-    <parent link="base_link"/>
-    <child link="camera_link"/>
-    <origin xyz="0.155 0 ${base_height/2 + 0.05}" rpy="0 0 0"/>
+  <joint name="depth_camera_joint" type="fixed">
+    <parent link="chassis_link"/>
+    <child link="depth_camera_link"/>
+    <origin xyz="0.155 0 ${chassis_height/2 + 0.015}" rpy="0 0 0"/>
   </joint>
-  <link name="camera_link_optical"></link>
-  <joint name="camera_optical_joint" type="fixed">
-    <parent link="camera_link"/>
-    <child link="camera_link_optical"/>
-    <origin xyz="0 0 0" rpy="${-pi/2} 0 ${-pi/2}"/>
-  </joint>
-  <gazebo reference="camera_link">
-    <material>Gazebo/Red</material>
-    <sensor name="camera" type="camera">
+  <gazebo reference="depth_camera_link">
+    <material>Gazebo/Silver</material>
+    <sensor name="depth_camera" type="depth_camera">
       <pose> 0 0 0 0 0 0 </pose>
+      <topic>depth_camera</topic>
       <visualize>true</visualize>
       <update_rate>10</update_rate>
       <camera>
-        <horizontal_fov>1.089</horizontal_fov>
+        <horizontal_fov>1.05</horizontal_fov>
         <image>
-          <format>R8G8B8</format>
-          <width>640</width>
-          <height>480</height>
+          <width>256</width>
+          <height>256</height>
+          <format>R_FLOAT32</format>
         </image>
         <clip>
-          <near>0.05</near>
-          <far>8.0</far>
+          <near>0.1</near>
+          <far>10.0</far>
         </clip>
       </camera>

File: dts_stack/urdf/ackermannRobot/gazebo_ackermann_control.xacro (robot description, xacro)
@@ -12,8 +12,8 @@
         <left_steering_joint>left_front_wheel_steering_joint</left_steering_joint>
         <right_steering_joint>right_front_wheel_steering_joint</right_steering_joint>
-        <kingpin_width>.18</kingpin_width>
+        <wheel_separation>.297</wheel_separation>
+        <kingpin_width>.28</kingpin_width>
         <steering_limit>0.5</steering_limit>
         <wheel_base>.33</wheel_base>
-        <wheel_separation>.297</wheel_separation>
         <wheel_radius>0.055</wheel_radius>
         <!-- Limits -->
@@ -25,10 +25,9 @@
         <topic>/cmd_vel</topic>
         <!-- Output -->
-        <odom_publish_frequency>100</odom_publish_frequency>
-        <odometry_frame>odom</odometry_frame>
-        <robot_base_frame>base_link</robot_base_frame>
-        <publish_odom>true</publish_odom>
-        <publish_odom_tf>true</publish_odom_tf>
-        <publish_wheel_tf>true</publish_wheel_tf>
+        <odom_publish_frequency>30</odom_publish_frequency>
+        <odom_topic>/odom</odom_topic>
+        <tf_topic>/tf</tf_topic>
+        <frame_id>/odom</frame_id>
+        <child_frame_id>/base_link</child_frame_id>
       </plugin>
     </gazebo>

File: dts_stack/urdf/ackermannRobot/imu.xacro (robot description, xacro)
@@ -13,12 +13,12 @@
       </geometry>
     </collision>
-    <xacro:inertial_box mass="0.1" x="0.075" y="0.075" z="0.02">
+    <xacro:box_inertial_w_origin mass="0.1" length="0.075" breadth="0.075" height="0.02">
     <origin xyz="0 0 0" rpy="0 0 0"/>
-  </xacro:inertial_box>
+  </xacro:box_inertial_w_origin>
   </link>
   <joint name="imu_joint" type="fixed">
-    <parent link="base_link"/>
+    <parent link="chassis_link"/>
     <child link="imu_link"/>
-    <origin xyz="-0.08 0 ${base_height/2 + 0.01}"/>
+    <origin xyz="-0.08 0 ${chassis_height/2 + 0.01}"/>
   </joint>
   <gazebo reference="imu_link">

File: dts_stack/urdf/ackermannRobot/inertial_macros.xacro (robot description, xacro)
@@ -3,5 +3,39 @@
     <!-- Specify some standard inertial calculations https://en.wikipedia.org/wiki/List_of_moments_of_inertia -->
     <!-- These make use of xacro's mathematical functionality -->
-    <xacro:macro name="inertial_sphere" params="mass radius *origin">
+    <xacro:macro name="box_inertial" params="mass length breadth height">
+        <inertial>
+            <mass value="${mass}" />
+            <inertia ixx="${(1/12) * mass * (breadth*breadth+height*height)}" ixy="0.0" ixz="0.0"
+                    iyy="${(1/12) * mass * (length*length+height*height)}" iyz="0.0"
+                    izz="${(1/12) * mass * (length*length+breadth*breadth)}" />
+        </inertial>
+    </xacro:macro>
+    <xacro:macro name="box_inertial_w_origin" params="mass length breadth height *origin">
+        <inertial>
+            <xacro:insert_block name="origin"/>
+            <mass value="${mass}" />
+            <inertia ixx="${(1/12) * mass * (breadth*breadth+height*height)}" ixy="0.0" ixz="0.0"
+                    iyy="${(1/12) * mass * (length*length+height*height)}" iyz="0.0"
+                    izz="${(1/12) * mass * (length*length+breadth*breadth)}" />
+        </inertial>
+    </xacro:macro>
+    <xacro:macro name="cylinder_inertial" params="mass length radius">
+        <inertial>
+            <mass value="${mass}" />
+            <inertia ixx="${(1/12) * mass * (3*radius*radius + length*length)}" ixy="0.0" ixz="0.0"
+                    iyy="${(1/12) * mass * (3*radius*radius + length*length)}" iyz="0.0"
+                    izz="${(1/2) * mass * (radius*radius)}" />
+        </inertial>
+    </xacro:macro>
+    <xacro:macro name="cylinder_inertial_w_origin" params="mass length radius *origin">
+        <inertial>
+            <xacro:insert_block name="origin"/>
+            <mass value="${mass}" />
+            <inertia ixx="${(1/12) * mass * (3*radius*radius + length*length)}" ixy="0.0" ixz="0.0"
+                    iyy="${(1/12) * mass * (3*radius*radius + length*length)}" iyz="0.0"
+                    izz="${(1/2) * mass * (radius*radius)}" />
+        </inertial>
+    </xacro:macro>
+    <xacro:macro name="sphere_inertial" params="mass radius *origin">
         <inertial>
             <xacro:insert_block name="origin"/>
@@ -12,21 +46,3 @@
         </inertial>
     </xacro:macro>
-    <xacro:macro name="inertial_box" params="mass x y z *origin">
-        <inertial>
-            <xacro:insert_block name="origin"/>
-            <mass value="${mass}" />
-            <inertia ixx="${(1/12) * mass * (y*y+z*z)}" ixy="0.0" ixz="0.0"
-                    iyy="${(1/12) * mass * (x*x+z*z)}" iyz="0.0"
-                    izz="${(1/12) * mass * (x*x+y*y)}" />
-        </inertial>
-    </xacro:macro>
-    <xacro:macro name="inertial_cylinder" params="mass length radius *origin">
-        <inertial>
-            <xacro:insert_block name="origin"/>
-            <mass value="${mass}" />
-            <inertia ixx="${(1/12) * mass * (3*radius*radius + length*length)}" ixy="0.0" ixz="0.0"
-                    iyy="${(1/12) * mass * (3*radius*radius + length*length)}" iyz="0.0"
-                    izz="${(1/2) * mass * (radius*radius)}" />
-        </inertial>
-    </xacro:macro>
 </robot>

File: dts_stack/urdf/ackermannRobot/lidar.xacro (robot description, xacro)
@@ -1,15 +1,16 @@
 <?xml version="1.0"?>
 <robot xmlns:xacro="http://www.ros.org/wiki/xacro" >
-  <link name="lidar_frame">
+  <!-- Define lidar constants -->
+  <xacro:property name="lidar_mass" value="0.01"/>
+  <xacro:property name="lidar_support_mass" value="0.01"/>
+  <xacro:property name="lidar_radius" value="0.025"/>
+  <xacro:property name="lidar_length" value="0.03"/>
+  <xacro:property name="lidar_support_breadth" value="0.06"/>
+  <xacro:property name="lidar_support_length" value="0.06"/>
+  <xacro:property name="lidar_support_height" value="0.06"/>
+  <link name="lidar_link">
     <visual>
       <geometry>
-        <cylinder radius="0.025" length="0.03"/>
-      </geometry>
-      <material name="black"/>
-    </visual>
-    <visual>
-      <origin xyz="0 0 -0.05"/>
-      <geometry>
-        <cylinder radius="0.01" length="0.1"/>
+        <cylinder radius="${lidar_radius}" length="${lidar_length}"/>
       </geometry>
       <material name="black"/>
@@ -17,21 +18,41 @@
     <collision>
       <geometry>
-        <cylinder radius="0.025" length="0.03"/>
+        <cylinder radius="${lidar_radius}" length="${lidar_length}"/>
       </geometry>
     </collision>
-    <xacro:inertial_cylinder mass="0.01" length="0.025" radius="0.03">
-      <origin xyz="0 0 0" rpy="0 0 0"/>
-    </xacro:inertial_cylinder>
+    <xacro:cylinder_inertial mass="${lidar_mass}" length="${lidar_length}" radius="${lidar_radius}"/>
+  </link>
+  <link name="lidar_support_link">
+    <visual>
+      <geometry>
+        <box size="${lidar_support_length} ${lidar_support_breadth} ${lidar_support_height}"/>
+      </geometry>
+      <material name="neon_blue"/>
+    </visual>
+    <collision>
+      <geometry>
+        <box size="${lidar_support_length} ${lidar_support_breadth} ${lidar_support_height}"/>
+      </geometry>
+    </collision>
+    <xacro:box_inertial mass="${lidar_mass}" length="${lidar_support_length}" breadth="${lidar_support_breadth}" height="${lidar_support_height}"/>
   </link>
   <joint name="lidar_joint" type="fixed">
-    <parent link="base_link"/>
-    <child link="lidar_frame"/>
-    <origin xyz="0.11 0 ${base_height/2 + 0.095}" rpy="0 0 ${pi}"/>
+    <parent link="lidar_support_link"/>
+    <child link="lidar_link"/>
+    <origin xyz="0 0 ${lidar_length/2 + lidar_support_height/2}" rpy="0 0 0"/>
   </joint>
-  <gazebo reference="lidar_frame">
+  <joint name="lidar_support_joint" type="fixed">
+    <parent link="chassis_link"/>
+    <child link="lidar_support_link"/>
+    <origin xyz="0.12 0 ${chassis_height/2 + lidar_support_height/2}" rpy="0 0 0"/>
+  </joint>
+  <gazebo reference="lidar_link">
     <material>Gazebo/Black</material>
-    <sensor name='lidar' type='gpu_lidar'>"
-      <pose relative_to='lidar_frame'>0 0 0 0 0 0</pose>
-      <topic>lidar</topic>
+    <sensor name='lidar_link' type='gpu_lidar'>"
+      <topic>scan_lidar</topic>
+      <ignition_frame_id>lidar_link</ignition_frame_id>
+      <pose relative_to='lidar_link'>0 0 0 0 0 0</pose>
+      <always_on>true</always_on>
+      <visualize>false</visualize>
       <update_rate>10</update_rate>
       <ray>
@@ -40,10 +61,10 @@
             <samples>640</samples>
             <resolution>1</resolution>
-            <min_angle>-1.396263</min_angle>
-            <max_angle>1.396263</max_angle>
+            <min_angle>-3.1416</min_angle>
+            <max_angle>3.1416</max_angle>
           </horizontal>
           <vertical>
             <samples>1</samples>
-            <resolution>0.01</resolution>
+            <resolution>0.1</resolution>
             <min_angle>0</min_angle>
             <max_angle>0</max_angle>
@@ -51,11 +72,9 @@
         </scan>
         <range>
-          <min>0.08</min>
+          <min>0.20</min>
           <max>10.0</max>
-          <resolution>0.01</resolution>
+          <resolution>0.1</resolution>
         </range>
       </ray>
-      <alwaysOn>1</alwaysOn>
-      <visualize>true</visualize>
     </sensor>
   </gazebo>

File: dts_stack/urdf/ackermannRobot/robot.urdf.xacro (robot description, xacro)
@@ -1,20 +1,15 @@
 <?xml version="1.0"?>
 <robot xmlns:xacro="http://www.ros.org/wiki/xacro"  name="robot">
-    <!-- ros2_control not implemented yet -->
-    <xacro:arg name="use_ros2_control" default="false"/>
-    <xacro:arg name="sim_mode" default="false"/>
+    <xacro:arg name="sim_mode" default="true"/>
     <!-- Robot model without sensors -->
     <xacro:include filename="robot_core.xacro" />
     <!-- Sensors -->
     <xacro:include filename="lidar.xacro" />
-    <xacro:include filename="camera.xacro" />
-<!--    <xacro:include filename="imu.xacro" /> -->
-<!--    <xacro:include filename="depth_camera.xacro" /> -->
+    <!-- <xacro:include filename="camera.xacro" />
+    <xacro:include filename="imu.xacro" />
+    <xacro:include filename="depth_camera.xacro" /> -->
     <!-- Controller -->
-    <xacro:if value="$(arg use_ros2_control)">
-        <xacro:include filename="ros2_control.xacro" />
+    <xacro:if value="$(arg sim_mode)">
+        <xacro:include filename="gazebo_ackermann_control.xacro" />
     </xacro:if>
-    <xacro:unless value="$(arg use_ros2_control)">
-        <xacro:include filename="gazebo_ackermann_control.xacro" />
-    </xacro:unless>
 </robot>
