Commit message: wip_with_gazebo

File: dts_stack/urdf/ackermannRobot/robot_core.xacro (robot description, xacro)
@@ -1,24 +1,29 @@
 <?xml version="1.0"?>
 <robot xmlns:xacro="http://www.ros.org/wiki/xacro" >
+  <xacro:arg name="wheel_diameter" default="0.11"/>
   <xacro:include filename="inertial_macros.xacro"/>
   <!-- Define robot constants -->
-  <xacro:property name="base_width" value="0.04"/>
-  <xacro:property name="base_length" value="0.56"/>
-  <xacro:property name="base_height" value="0.07"/>
-  <xacro:property name="base_mass" value="0.07"/>
-  <xacro:property name="wheel_radius" value="0.055"/>
+  <xacro:property name="wheel_mass" value="0.2"/>
+  <xacro:property name="chassis_mass" value = "1.5"/>
+  <xacro:property name="axle_mass" value="0.2"/>
+  <xacro:property name="bumper_mass" value = "0.2"/>
+  <xacro:property name="wheel_radius" value="${$(arg wheel_diameter)/2}"/>
   <xacro:property name="wheel_width" value="0.045"/>
-  <xacro:property name="wheel_mass" value="0.05"/>
-  <xacro:property name="wheel_offset_x_front" value="0.17"/>
-  <xacro:property name="wheel_offset_x_rear" value="0.16"/>
-  <xacro:property name="wheel_offset_y" value="0.1485"/>
-  <material name="blue">
-    <color rgba="0 0 0.8 1"/>
-  </material>
+  <xacro:property name="steering_kingpin_mass" value = "0.001"/>
+  <xacro:property name="steering_kingpin_length" value = "0.014"/>
+  <xacro:property name="steering_kingpin_radius" value = "0.001"/>
+  <xacro:property name="wheelbase_length" value="0.33"/>
+  <xacro:property name="chassis_breadth" value = "0.18"/>
+  <xacro:property name="chassis_length" value = "${wheelbase_length}"/>
+  <xacro:property name="bumper_horiz_length" value = "0.1"/>
+  <xacro:property name="bumper_vert_length" value = "0.045"/>
+  <xacro:property name="bumper_thickness" value = "0.01"/>
+  <xacro:property name="overall_body_length" value = "${wheelbase_length+2*bumper_horiz_length}"/>
+  <xacro:property name="chassis_height" value = "0.08"/>
+  <xacro:property name="front_wheelbase_breadth" value="0.21"/>
+  <xacro:property name="rear_wheelbase_breadth" value="0.21"/>
+  <xacro:property name="axle_radius" value="0.005"/>
   <material name="black">
     <color rgba="0 0 0 1"/>
-  </material>
-  <material name="white">
-    <color rgba="1 1 1 1"/>
   </material>
   <material name="lime">
@@ -28,199 +33,271 @@
     <color rgba="0.75 0.75 0.75 1"/>
   </material>
-  <material name="orange">
-    <color rgba="1 0.3 0.1 1"/>
-  </material>
-  <material name="red">
-    <color rgba="1 0 0 1"/>
+  <material name="neon_blue">
+    <color rgba="0.01 0.54 1 1"/>
   </material>
   <!-- Robot Base -->
-  <link name="base_link">
-  <visual>
-    <geometry>
-      <box size="${base_length} ${base_width} ${base_height}"/>
-    </geometry>
+  <link name="base_link"/>
+  <link name="chassis_link">
+    <visual>
+      <origin xyz="0 0 0" rpy="0 0 0"/>
+      <geometry>
+        <box size="${chassis_length} ${chassis_breadth} ${chassis_height}"/>
+      </geometry>
       <material name="lime"/>
-  </visual>
-  <collision>
-    <geometry>
-      <box size="${base_length} ${base_width} ${base_height}"/>
-    </geometry>
-  </collision>
-  <xacro:inertial_box mass="${base_mass}" x="${base_length}" y="${base_width}" z="${base_height}">
-    <origin xyz="${base_length/2} 0 ${base_height/2}" rpy="0 0 0"/>
-  </xacro:inertial_box>
-  </link>
-  <!-- Robot Footprint -->
-  <link name="base_footprint"/>
-  <joint name="base_joint" type="fixed">
+    </visual>
+    <collision>
+      <geometry>
+        <box size="${chassis_length} ${chassis_breadth} ${chassis_height}"/>
+      </geometry>
+    </collision>
+    <xacro:box_inertial mass="${chassis_mass}" length="${chassis_length}" breadth="${chassis_breadth}" height="${chassis_height}"/>
+  </link>
+  <joint name="chassis_joint" type="fixed">
     <parent link="base_link"/>
-    <child link="base_footprint"/>
-    <origin xyz="0.0 0.0 ${-wheel_radius}" rpy="0 0 0"/>
-  </joint>
+    <child link="chassis_link"/>
+    <origin rpy="0 0 0" xyz="0 0 ${wheel_radius+chassis_height/2}"/>
+  </joint>
+  <link name="bumper_link">
+    <visual>
+      <origin xyz="${chassis_length/2 + bumper_horiz_length/2} 0 ${-chassis_height/2+bumper_thickness/2}" rpy="0 0 0"/>
+      <geometry>
+        <box size="${bumper_horiz_length} ${chassis_breadth} ${bumper_thickness}"/>
+      </geometry>
+      <material name="black"/>
+    </visual>
+    <visual>
+      <origin xyz="${-chassis_length/2 - bumper_horiz_length/2} 0 ${-chassis_height/2+bumper_thickness/2}" rpy="0 0 0"/>
+      <geometry>
+        <box size="${bumper_horiz_length} ${chassis_breadth} ${bumper_thickness}"/>
+      </geometry>
+      <material name="black"/>
+    </visual>
+    <visual>
+      <origin xyz="${chassis_length/2 + bumper_horiz_length - bumper_thickness/2} 0 ${-chassis_height/2+bumper_vert_length/2}" rpy="0 0 0"/>
+      <geometry>
+        <box size="${bumper_thickness} ${chassis_breadth} ${bumper_vert_length}"/>
+      </geometry>
+      <material name="black"/>
+    </visual>
+    <visual>
+      <origin xyz="${-chassis_length/2 - bumper_horiz_length + bumper_thickness/2} 0 ${-chassis_height/2+bumper_vert_length/2}" rpy="0 0 0"/>
+      <geometry>
+        <box size="${bumper_thickness} ${chassis_breadth} ${bumper_vert_length}"/>
+      </geometry>
+      <material name="black"/>
+    </visual>
+    <collision>
+      <geometry>
+        <box size="${overall_body_length} ${chassis_breadth} ${bumper_vert_length}"/>
+      </geometry>
+    </collision>
+    <xacro:box_inertial mass="${bumper_mass}" length="${overall_body_length}" breadth="${chassis_breadth}" height="${bumper_vert_length}"/>
+  </link>
+  <joint name="bumper_joint" type="fixed">
+    <parent link="chassis_link"/>
+    <child link="bumper_link"/>
+    <origin rpy="0 0 0" xyz="0 0 0"/>
+  </joint>
+  <!-- Rear axle -->
+  <link name="rear_axle_link">
+    <visual>
+      <geometry>
+        <cylinder length="${rear_wheelbase_breadth}" radius="${axle_radius}"/>
+      </geometry>
+      <material name="silver"/>
+    </visual>
+    <collision>
+      <geometry>
+        <cylinder length="${rear_wheelbase_breadth}" radius="${axle_radius}"/>
+      </geometry>
+    </collision>
+    <xacro:cylinder_inertial mass="${axle_mass}" radius="${axle_radius}" length="${rear_wheelbase_breadth}"/>
+  </link>
+  <joint name="rear_axle_joint" type="fixed">
+    <parent link="chassis_link"/>
+    <child link="rear_axle_link"/>
+    <origin xyz="${-wheelbase_length/2} 0 ${-chassis_height/2}" rpy="${-pi/2} 0 0"/>
+  </joint>
+  <!-- Left rear wheel -->
+  <link name="left_rear_wheel_link">
+    <visual>
+      <geometry>
+        <cylinder length="${wheel_width}" radius="${wheel_radius}"/>
+      </geometry>
+      <material name="black">
+        <color rgba="0 0 0 1"/>
+      </material>
+    </visual>
+    <collision>
+      <geometry>
+        <cylinder length="${wheel_width}" radius="${wheel_radius}"/>
+      </geometry>
+    </collision>
+    <xacro:cylinder_inertial mass="${wheel_mass}" radius="${wheel_radius}" length="${wheel_width}"/>
+  </link>
+  <joint name="left_rear_wheel_joint" type="continuous">
+    <axis xyz="0 0 1"/>
+    <parent link="rear_axle_link"/>
+    <child link="left_rear_wheel_link"/>
+    <origin xyz="0 0 ${rear_wheelbase_breadth/2+wheel_width/2}" rpy="0 0 0" />
+    <limit effort="10000" velocity="500" />
+  </joint>
+  <gazebo reference="left_rear_wheel_link">
+    <material>Gazebo/DarkGrey</material>
+  </gazebo>
   <!-- Right rear wheel -->
   <link name="right_rear_wheel_link">
     <visual>
-      <origin rpy="${-pi/2} 0 0" xyz="0 0 0"/>
-      <geometry>
-        <cylinder length="${wheel_width}" radius="${wheel_radius}"/>
-      </geometry>
-      <material name="black"/>
-    </visual>
-    <collision>
-      <origin rpy="${-pi/2} 0 0" xyz="0 0 0"/>
-      <geometry>
-        <cylinder length="${wheel_width}" radius="${wheel_radius}"/>
-      </geometry>
-    </collision>
-    <xacro:inertial_cylinder mass="${wheel_mass}" length="${wheel_width}" radius="${wheel_radius}">
-      <origin xyz="0 0 0" rpy="0 0 0"/>
-    </xacro:inertial_cylinder>
-    <velocity_decay/>
-  </link>
-  <gazebo reference="right_rear_wheel_link">
-    <material>Gazebo/Blue</material>
-    <mu1>10.5</mu1>
-    <mu2>1.0</mu2>
-    <fdir1>0 0 1</fdir1>
-    <gravity>true</gravity>
+      <geometry>
+        <cylinder length="${wheel_width}" radius="${wheel_radius}"/>
+      </geometry>
+      <material name="black">
+        <color rgba="0 0 0 1"/>
+      </material>
+    </visual>
+    <collision>
+      <geometry>
+        <cylinder length="${wheel_width}" radius="${wheel_radius}"/>
+      </geometry>
+    </collision>
+    <xacro:cylinder_inertial mass="${wheel_mass}" radius="${wheel_radius}" length="${wheel_width}"/>
+  </link>
+  <joint name="right_rear_wheel_joint" type="continuous">
+    <axis xyz="0 0 1"/>
+    <parent link="rear_axle_link"/>
+    <child link="right_rear_wheel_link"/>
+    <origin xyz="0 0 ${-rear_wheelbase_breadth/2-wheel_width/2}" rpy="0 0 0"/>
+    <limit effort="10000" velocity="500" />
+  </joint>
+  <gazebo reference="right_front_wheel_link">
+    <material>Gazebo/DarkGrey</material>
   </gazebo>
-  <joint name="right_rear_wheel_joint" type="revolute">
-    <parent link="base_link"/>
-    <child link="right_rear_wheel_link"/>
-    <origin rpy="0 0 0" xyz="${-wheel_offset_x_rear} ${-wheel_offset_y} 0"/>
-    <axis xyz="0 1 0"/>
-    <limit effort="25" lower="-1.79769e+308" upper="1.79769e+308" velocity="100"/>
-    <dynamics damping="0.0" friction="0.0"/>
-  </joint>
-  <!-- Left rear wheel -->
-  <link name="left_rear_wheel_link">
-    <visual>
-      <origin rpy="${-pi/2} 0 0" xyz="0 0 0"/>
-      <geometry>
-        <cylinder length="${wheel_width}" radius="${wheel_radius}"/>
-      </geometry>
-      <material name="black"/>
-    </visual>
-    <collision>
-      <origin rpy="${-pi/2} 0 0" xyz="0 0 0"/>
-      <geometry>
-        <cylinder length="${wheel_width}" radius="${wheel_radius}"/>
-      </geometry>
-    </collision>
-    <xacro:inertial_cylinder mass="${wheel_mass}" length="${wheel_width}" radius="${wheel_radius}">
-      <origin xyz="0 0 0" rpy="0 0 0"/>
-    </xacro:inertial_cylinder>
-    <velocity_decay/>
-  </link>
-  <gazebo reference="left_rear_wheel_link">
-    <material>Gazebo/Blue</material>
-    <mu1>10.5</mu1>
-    <mu2>1.0</mu2>
-    <fdir1>0 0 1</fdir1>
-    <gravity>true</gravity>
-  </gazebo>
-  <joint name="left_rear_wheel_joint" type="revolute">
-    <parent link="base_link"/>
-    <child link="left_rear_wheel_link"/>
-    <origin rpy="0 0 0" xyz="${-wheel_offset_x_rear} ${wheel_offset_y} 0"/>
-    <axis xyz="0 1 0"/>
-    <limit effort="25" lower="-1.79769e+308" upper="1.79769e+308" velocity="100"/>
-    <dynamics damping="0.0" friction="0.0"/>
-  </joint>
-  <!-- Left front wheel and steering -->
+  <!-- Front axle -->
+  <link name="front_axle_link">
+    <visual>
+      <geometry>
+        <cylinder length="${front_wheelbase_breadth}" radius="${axle_radius}"/>
+      </geometry>
+      <material name="silver"/>
+    </visual>
+    <collision>
+      <geometry>
+        <cylinder length="${front_wheelbase_breadth}" radius="${axle_radius}"/>
+      </geometry>
+    </collision>
+    <xacro:cylinder_inertial mass="${axle_mass}" radius="${axle_radius}" length="${front_wheelbase_breadth}"/>
+  </link>
+  <joint name="front_axle_joint" type="fixed">
+    <parent link="chassis_link"/>
+    <child link="front_axle_link"/>
+    <origin xyz="${wheelbase_length/2} 0 ${-chassis_height/2}" rpy="${-pi/2} 0 0"/>
+  </joint>
+  <!-- Left front wheel steering -->
   <link name="left_front_wheel_steering_link">
-    <inertial>
-      <mass value="0.005"/>
-      <inertia ixx=".0000018" ixy="0" ixz="0" iyy=".0000018" iyz="0" izz=".0000018"/>
-    </inertial>
+    <visual>
+      <geometry>
+        <cylinder length="${steering_kingpin_length}" radius="${steering_kingpin_radius}"/>
+      </geometry>
+      <material name="black"/>
+    </visual>
+    <collision>
+      <geometry>
+        <cylinder length="${steering_kingpin_length}" radius="${steering_kingpin_radius}"/>
+      </geometry>
+    </collision>
+    <xacro:cylinder_inertial mass="${steering_kingpin_mass}" radius="${steering_kingpin_radius}" length="${steering_kingpin_length}"/>
   </link>
   <joint name="left_front_wheel_steering_joint" type="revolute">
-    <parent link="base_link"/>
+    <axis xyz="0 0 1"/>
+    <limit lower="${-pi/3}" upper="${pi/3}" effort="1000000" velocity="500"/>
+    <parent link="front_axle_link"/>
     <child link="left_front_wheel_steering_link"/>
-    <origin rpy="0 0 0" xyz="${wheel_offset_x_front} ${wheel_offset_y} 0"/>
-    <axis xyz="0 0 1"/>
-    <limit effort="25" lower="-0.6" upper="0.6" velocity="1.0"/>
-  </joint>
+    <origin xyz="0 0 ${front_wheelbase_breadth/2-steering_kingpin_radius}" rpy="${pi/2} 0 0" />
+  </joint>
+  <!-- <gazebo reference="left_front_wheel_steering_joint">
+    <material>Gazebo/DarkGrey</material>
+    <springStiffness>0.1</springStiffness>
+    <springReference>0</springReference>
+    <implicitSpringDamper>true</implicitSpringDamper>
+    <fudgeFactor>0</fudgeFactor>
+  </gazebo> -->
+  <!-- Left front wheel -->
   <link name="left_front_wheel_link">
     <visual>
-      <origin rpy="${-pi/2} 0 0" xyz="0 0 0"/>
-      <geometry>
-        <cylinder length="${wheel_width}" radius="${wheel_radius}"/>
-      </geometry>
-      <material name="black"/>
-    </visual>
-    <collision>
-      <origin rpy="${-pi/2} 0 0" xyz="0 0 0"/>
-      <geometry>
-        <cylinder length="${wheel_width}" radius="${wheel_radius}"/>
-      </geometry>
-    </collision>
-    <xacro:inertial_cylinder mass="${wheel_mass}" length="${wheel_width}" radius="${wheel_radius}">
-      <origin xyz="0 0 0" rpy="0 0 0"/>
-    </xacro:inertial_cylinder>
-    <velocity_decay/>
-  </link>
-  <gazebo reference="left_front_wheel_link">
-    <material>Gazebo/Blue</material>
-    <mu1>10.5</mu1>
-    <mu2>1.0</mu2>
-    <fdir1>0 0 1</fdir1>
-    <gravity>true</gravity>
-  </gazebo>
-  <joint name="left_front_wheel_joint" type="revolute">
+      <geometry>
+        <cylinder length="${wheel_width}" radius="${wheel_radius}"/>
+      </geometry>
+      <material name="black"/>
+    </visual>
+    <collision>
+      <geometry>
+        <cylinder length="${wheel_width}" radius="${wheel_radius}"/>
+      </geometry>
+    </collision>
+    <xacro:cylinder_inertial mass="${wheel_mass}" radius="${wheel_radius}" length="${wheel_width}"/>
+  </link>
+  <joint name="left_front_wheel_joint" type="continuous">
+    <axis xyz="0 0 1"/>
     <parent link="left_front_wheel_steering_link"/>
     <child link="left_front_wheel_link"/>
-    <origin rpy="0 0 0" xyz="0 0 0"/>
-    <axis xyz="0 1 0"/>
-    <limit effort="25" lower="-1.79769e+308" upper="1.79769e+308" velocity="100"/>
-    <dynamics damping="0.0" friction="0.0"/>
-  </joint>
-  <!-- Right front wheel and steering -->
+    <origin xyz="0 ${steering_kingpin_radius+wheel_width/2} 0" rpy="${-pi/2} 0 0"/>
+    <limit effort="10000" velocity="500" />
+  </joint>
+  <gazebo reference="left_front_wheel_link">
+    <material>Gazebo/DarkGrey</material>
+  </gazebo>
+  <!-- Right front wheel steering -->
   <link name="right_front_wheel_steering_link">
-    <inertial>
-      <mass value="0.005"/>
-      <inertia ixx=".0000018" ixy="0" ixz="0" iyy=".0000018" iyz="0" izz=".0000018"/>
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